File: hardware/digi/audio_codec.kicad_sch (KiCad schematic)
At the start: 15 parts, among them IC1 ES8311, J2 IN, J3 OUT, U3 TL072

Commit message: renders, etc
Parts:
- added L2: 180r-100M, Inductor_SMD:L_0805_2012Metric, symbol Device:L_Ferrite
- added TP7: AUDIO_IN, TestPoint:TestPoint_Pad_D2.5mm, symbol Connector:TestPoint
- added TP8: AUDIO_VMID, TestPoint:TestPoint_Pad_D2.5mm, symbol Connector:TestPoint
- C26, C27, C28, C29, C30, C31, C32, C33: footprint (none) -> Capacitor_SMD:C_0402_1005Metric
- IC1: footprint QFN40P300X300X60-21N -> ES8311:QFN40P300X300X60-21N
- J2, J3: footprint (none) -> PJ301M-2-B:Jack_3.5mm_QingPu_WQP-PJ301M-12_Vertical
- R11, R12, R13: footprint (none) -> Resistor_SMD:R_0402_1005Metric
- U3: footprint (none) -> TL072:D8_TEX_STM
Connections:
- net +3V3: now also L2.1; no longer C29.1, IC1.11 (AVDD)
- net AUDIO_VMID: now also C26.1, IC1.16 (VMID), TP8.1
- net at C32.2, IC1.18 (MIC1P/DMIC_SDA), R13.1: now also TP7.1
- new net AVDD: C29.1, IC1.11 (AVDD), L2.2
Other:
- title: (none) -> AUDIO CODEC
- moved on the sheet: C29
