File: hardware/digi/digi.kicad_sch (KiCad schematic)
At the start: 16 parts, among them J1 USB_B_Micro, U2 FT4222HQ, Y1 12MHz

Commit message: renders, etc
Parts:
- added C36: 100n, Capacitor_SMD:C_0402_1005Metric, symbol Device:C
- added R14: DNP, Resistor_SMD:R_0805_2012Metric_Pad1.20x1.40mm_HandSolder, symbol Device:R
- added R21: 10k, Resistor_SMD:R_0805_2012Metric, symbol Device:R
- added R22: 2.2k, Resistor_SMD:R_0402_1005Metric, symbol Device:R
- added R23: 0, Resistor_SMD:R_0402_1005Metric, symbol Device:R
- added TP5: VBUS, TestPoint:TestPoint_Pad_D2.5mm, symbol Connector:TestPoint
- C16, C17: value C -> 20p; footprint (none) -> Capacitor_SMD:C_0402_1005Metric
- C18, C19, C20, C21, C22, C23, C24, C25: footprint (none) -> Capacitor_SMD:C_0402_1005Metric
- J1: footprint (none) -> MICROXNJ:SHOUHAN_MICROXNJ
- L1: footprint (none) -> Inductor_SMD:L_0805_2012Metric
- R10, R9: footprint (none) -> Resistor_SMD:R_0402_1005Metric
- Y1: value 12MHz -> 12MHz - X322512MSB4SI; footprint (none) -> Crystal:Crystal_SMD_3225-4Pin_3.2x2.5mm
Connections:
- net +3V3: now also R21.2, R22.2
- net GND: now also C36.2, R14.1, R23.2
- net VBUS: now also TP5.1
- net USB_D-: now reaches J1.2 (D-), U2.23 (DP)
- net USB_D+: now reaches J1.3 (D+), U2.22 (DM)
- net at J1.4 (ID): now also C36.1, R23.1
- net at U2.3 (~{RESET}): now also R22.1
- net at U2.4 (DCNF0): now also U2.5 (DCNF1), R14.2, R21.1
- net ICE_SPI_MISO renamed ICE_SPI1_MISO
- net ICE_SPI_MOSI renamed ICE_SPI1_MOSI
- net ICE_SPI_SCK renamed ICE_SPI1_SCK
- net USB_SPI_CS renamed USB_SPI1_CS
- no-connect marks 2 -> 9
Other:
- moved on the sheet: C16, C17
