File: hardware/digi/ice40up5k.kicad_sch (KiCad schematic)
At the start: 29 parts, among them SW1 RESET_SW, U1 ICE40UP5K-SG48ITR

Commit message: renders, etc
Parts:
- added D10: LED_G, LED_SMD:LED_0805_2012Metric, symbol Device:LED
- added D11: LED_B, LED_SMD:LED_0805_2012Metric, symbol Device:LED
- added D9: LED_R, LED_SMD:LED_0805_2012Metric, symbol Device:LED
- added R28, R29, R30: 100, Resistor_SMD:R_0402_1005Metric, symbol Device:R
- added TP6: RESET, TestPoint:TestPoint_Pad_D2.5mm, symbol Connector:TestPoint
- C1, C10, C11, C12, C13, C14, C15, C2, C3, C4, C5, C6, C7, C8, C9: footprint (none) -> Capacitor_SMD:C_0402_1005Metric
- D1: value D -> 1N4148; footprint (none) -> Diode_SMD:D_SOD-323
- D2: footprint (none) -> LED_SMD:LED_0805_2012Metric
- JP1, JP2: footprint (none) -> Connector_PinHeader_2.54mm:PinHeader_1x02_P2.54mm_Vertical
- R1, R8: footprint (none) -> Resistor_SMD:R_0402_1005Metric
- R2, R3, R4, R5, R6: value 1 -> 0; footprint (none) -> Resistor_SMD:R_0402_1005Metric
- R7: footprint (none) -> Resistor_SMD:R_0805_2012Metric
- SW1: footprint (none) -> TS-1088-AR02016:SW_TS-1088-AR02016
Connections:
- net +3V3: now also D10.2 (A), D11.2 (A), D9.2 (A); no longer R5.1
- net CRESET: now also TP6.1
- net ENCODER_1_A: no longer U1.26 (IOT_39a)
- net ENCODER_2_A: no longer U1.31 (IOT_42b)
- net ICE_I2S_DIN: now also U1.48 (IOB_4a); no longer U1.45 (IOB_5b)
- net ICE_I2S_DOUT: now also U1.44 (IOB_3b_G6); no longer U1.48 (IOB_4a)
- net ICE_I2S_WS: now also U1.38 (IOT_50b); no longer U1.44 (IOB_3b_G6)
- net ICE_LED_0: now reaches U1.39 (RGB0)
- net ICE_LED_0: now also R30.1
- net ICE_LED_1: now reaches U1.40 (RGB1)
- net ICE_LED_1: now also R29.1
- net ICE_LED_2: now reaches U1.41 (RGB2)
- net ICE_LED_2: now also R28.1
- net IOT_51a: now reaches U1.42 (IOT_51a)
- net NEOPIXEL_DIN: now reaches U1.43 (IOT_49a)
- net IOB_18a: now reaches U1.10 (IOB_18a)
- net IOB_20a: now reaches U1.11 (IOB_20a)
- net IOB_22a: now reaches U1.12 (IOB_22a)
- net IOB_24a: now reaches U1.13 (IOB_24a)
- net IOB_29b: now reaches U1.19 (IOB_29b)
- net IOB_25b_G3: now reaches U1.20 (IOB_25b_G3)
- net IOB_23b: now reaches U1.21 (IOB_23b)
- net IOB_13b: now reaches U1.6 (IOB_13b)
- net IOB_16a: now reaches U1.9 (IOB_16a)
- net ICE_SPI1_MISO: now reaches U1.2 (IOB_6a)
- net ICE_SPI1_SCK: now reaches U1.3 (IOB_9b)
- net ICE_SPI1_MOSI: now reaches U1.4 (IOB_8a)
- net ICE_SPI_MISO renamed ICE_SPI0_MISO
- net ICE_SPI_MOSI renamed ICE_SPI0_MOSI
- net ICE_SPI_SCK renamed ICE_SPI0_SCK
- net PSRAM_SPI_CS renamed IOB_31b
- net USB_SPI_CS renamed PSRAM_SPI0_CS
- new net: D11.1 (K), R30.2
- new net: D9.1 (K), R28.2
- new net: D10.1 (K), R29.2
- new net +1V8: R5.1
- new net ENCODER_1_B: U1.26 (IOT_39a)
- new net ENCODER_2_B: U1.31 (IOT_42b)
- new net USB_SPI1_CS: U1.45 (IOB_5b)
Other:
- note added: "INDICATOR LEDS"
- note removed: "FINSIH USB-SPI"
- note removed: "FIX AUDIO OUT"
- note removed: "LDOs - 3.3, 1.2, 1.8"
- note removed: "TODO"
- note removed: "encoders other control inputs Control feedback"
- title: (none) -> ICE40UP5K
