File: hardware/digi/inputs.kicad_sch (KiCad schematic)
At the start: 11 parts, among them SW2 Encoder1, SW3 Encoder2, SW4 SW_SPDT, SW5 SW_SPDT, SW6 SW_SPDT

Commit message: renders, etc
Parts:
- added C37, C38, C54, C55: 100n, Capacitor_SMD:C_0402_1005Metric, symbol Device:C_Small
- added D12, D6, D7, D8: NeoPixel_THT, LED_THT:LED_D5.0mm-4_RGB_Staggered_Pins, symbol LED:NeoPixel_THT
- R15, R16, R17, R18, R19, R20: footprint (none) -> Resistor_SMD:R_0805_2012Metric
- SW2, SW3: footprint (none) -> Rotary_Encoder:RotaryEncoder_Alps_EC11E-Switch_Vertical_H20mm_MountingHoles
- SW4, SW5, SW6: footprint (none) -> Connector_PinHeader_2.54mm:PinHeader_1x03_P2.54mm_Vertical
Connections:
- net +3V3: now also C37.1, C38.1, C54.1, C55.1, D12.3 (VDD), D6.3 (VDD), D7.3 (VDD), D8.3 (VDD)
- net ENCODER_1_A: no longer R18.2, SW2.B
- net ENCODER_2_A: no longer R20.2, SW3.B
- net GND: now also C37.2, C38.2, C54.2, C55.2, D12.2 (GND), D6.2 (GND), D7.2 (GND), D8.2 (GND)
- new net: D6.1 (DOUT), D7.4 (DIN)
- new net: D12.4 (DIN), D8.1 (DOUT)
- new net: D7.1 (DOUT), D8.4 (DIN)
- new net ENCODER_1_B: R18.2, SW2.B
- new net ENCODER_2_B: R20.2, SW3.B
- new net NEOPIXEL_DIN: D6.4 (DIN)
- no-connect marks 0 -> 1
Other:
- note added: "ROTARY ENCODER INDICATOR NEOPIXELS"
- title: (none) -> CONTROLS
- moved on the sheet: SW4, SW5, SW6
