File: hardware/digi/sdram.kicad_sch (KiCad schematic)
At the start: 3 parts, among them IC2 APS6404L-SQN-SN

Commit message: renders, etc
Parts:
- added C60: 100n, Capacitor_SMD:C_0402_1005Metric, symbol Device:C
- added C61: 4.7u, Capacitor_SMD:C_0402_1005Metric, symbol Device:C
- added TP10: FLASH_CLK, TestPoint:TestPoint_Pad_D2.5mm, symbol Connector:TestPoint
- added TP9: FLASH_SDA, TestPoint:TestPoint_Pad_D2.5mm, symbol Connector:TestPoint
- added U7: AT24C256C-SSHL-T, AT24C256C-SSHL-T:SOIC127P600X175-8N, symbol AT24C256C-SSHL-T:AT24C256C-SSHL-T
- C34, C35: footprint (none) -> Capacitor_SMD:C_0402_1005Metric
- IC2: footprint SOIC127P600X175-8N -> APS6404L-SQN-SN:SOIC127P600X175-8N
Connections:
- net GND: now also C60.2, C61.2, U7.1 (A0), U7.2 (A1), U7.3 (A2), U7.4 (GND), U7.7 (WP)
- net ICE_SPI_MISO renamed ICE_SPI0_MISO
- net ICE_SPI_MOSI renamed ICE_SPI0_MOSI
- net ICE_SPI_SCK renamed ICE_SPI0_SCK
- net PSRAM_SPI_CS renamed PSRAM_SPI0_CS
- new net +3V3: C60.1, C61.1, U7.8 (VCC)
- new net ICE_I2C_CLK: TP10.1, U7.6 (SCL)
- new net ICE_I2C_SDA: TP9.1, U7.5 (SDA)
Other:
- note added: "FLASH"
- title: (none) -> MEMORY
